File: Test/Test.kicad_sch (KiCad schematic)
At the start: 4 parts, among them J1 Conn_01x20, J2 Conn_01x20, J3 Conn_01x03, U1 Pico

Commit message: Updated footprints to their correct types -  Updated 'Test' project to use updated footprint
Parts:
- J1, J2: footprint Connector_PinSocket_1.00mm:PinSocket_1x20_P1.00mm_Vertical -> Connector_PinSocket_2.54mm:PinSocket_1x20_P2.54mm_Vertical
- J3: footprint Connector_PinSocket_1.00mm:PinSocket_1x03_P1.00mm_Vertical -> Connector_PinSocket_2.54mm:PinSocket_1x03_P2.54mm_Vertical
Changed lines of the file:
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@@
       (effects (font (size 1.27 1.27)))
     )
-    (property "Footprint" "Connector_PinSocket_1.00mm:PinSocket_1x20_P1.00mm_Vertical" (at 54.61 76.2 0)
+    (property "Footprint" "Connector_PinSocket_2.54mm:PinSocket_1x20_P2.54mm_Vertical" (at 54.61 76.2 0)
       (effects (font (size 1.27 1.27)) hide)
     )
@@
       (effects (font (size 1.27 1.27)) (justify left))
     )
-    (property "Footprint" "Connector_PinSocket_1.00mm:PinSocket_1x20_P1.00mm_Vertical" (at 144.78 76.2 0)
+    (property "Footprint" "Connector_PinSocket_2.54mm:PinSocket_1x20_P2.54mm_Vertical" (at 144.78 76.2 0)
       (effects (font (size 1.27 1.27)) hide)
     )
@@
       (effects (font (size 1.27 1.27)) (justify left))
     )
-    (property "Footprint" "Connector_PinSocket_1.00mm:PinSocket_1x03_P1.00mm_Vertical" (at 101.6 116.84 0)
+    (property "Footprint" "Connector_PinSocket_2.54mm:PinSocket_1x03_P2.54mm_Vertical" (at 101.6 116.84 0)
       (effects (font (size 1.27 1.27)) hide)
     )
